Commit message: Added lidar simulation and ROS2 Humble fixes

File: description/gazebo_control.xacro (robot description, xacro)
@@ -2,20 +2,4 @@
 <robot xmlns:xacro="http://www.ros.org/wiki/xacro">
     <gazebo>
-   plugin name="diff_drive" filename="libgazebo_ros_diff_drive.so">
-    <!-- Wheel information -->
-    <left_joint>left_wheel_joint</left_joint>
-    <right_joint>right_wheel_joint</right_joint>
-    <wheel_separation>0.35</wheel_separation>
-    <wheel_diameter>0.1</wheel_diameter>
-    <!-- Limits -->
-    <max_wheel_torque>200</max_wheel_torque>
-    <max_wheel_acceleration>10.0</max_wheel_acceleration>
-    <!-- Output -->
-    <odometry_frame>odom</odometry_frame>
-    <robot_base_frame>base_link</robot_base_frame>
-    <publish_odom>true</publish_odom>
-    <publish_odom_tf>true</publish_odom_tf>
-    <publish_wheel_tf>true</publish_wheel_tf>
-     </plugin>
     </gazebo>
 </robot>

File: description/robot.urdf.xacro (robot description, xacro)
@@ -1,4 +1,6 @@
 <?xml version="1.0"?>
 <robot xmlns:xacro="http://www.ros.org/wiki/xacro" name="robot">
-      <xacro:include filename ="robot_core.xacro"/>
+    <xacro:include filename="robot_core.xacro"/>
+    <xacro:include filename="lidar.xacro"/>
+    <xacro:lidar/>
 </robot>

File: description/robot_core.xacro (robot description, xacro)
@@ -15,4 +15,7 @@
         <color rgba="0 0 0 1"/>
     </material>
+    <material name="red">
+    <color rgba="1 0 0 1"/>
+</material>
     <!-- Base Link -->
     <link name="base_link">
